File: PCB/gantry-controller-prototype-DUE/Arduino_DUE_Connections.sch (KiCad schematic (older format))
At the start: 68 parts, among them J1 Conn_01x07, M4 Arduino_DUE_Shield_TEMP, T11 1755503, T12 1755503, T13 1740369, T14 1740369, T15 1740369, T16 1740369, T17 1740369, T20 5033981892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

Commit message: Fab files and edits
made some changes to the circuit, added pullups to OE pins on 74 devices and tied mosfet drivers to GND, added fab files
Parts:
- added R42, R43, R44, R45: RC0402FR-071KL, AVR-KiCAD-Lib-Resistors:R0402, symbol growbox-KiCAD-Resistors:RC0402FR-071KL
Connections:
- net +3V3: now also R42.2, R43.2, R44.2, R45.2
- net GND: now also U6.2 (ADDR)
- net at M4.D37, U7.1 (1OE): now also R44.1
- net at M4.D13, U7.24 (4OE): now also R42.1
- net at M4.D12, U7.25 (3OE): now also R43.1
- net at M4.D35, U7.48 (2OE): now also R45.1
Other:
- moved on the sheet: L4
