File: PCB/gantry-controller-prototype-DUE/EStop_Lights.sch (KiCad schematic (older format))
At the start: 35 parts, among them Q1 IRLML6346TRPBF, Q2 IRLML6346TRPBF, Q3 IRLML6346TRPBF, Q4 IRLML6346TRPBF, T18 1755574, U1 SN74AHCT125RGYR, U2 ZXGD3009E6TA, U3 ZXGD3009E6TA, U4 ZXGD3009E6TA, U5 ZXGD3009E6TA

Commit message: Fab files and edits
made some changes to the circuit, added pullups to OE pins on 74 devices and tied mosfet drivers to GND, added fab files
Parts:
- added R38, R39, R40, R41: RC0402FR-071KL, AVR-KiCAD-Lib-Resistors:R0402, symbol growbox-KiCAD-Resistors:RC0402FR-071KL
Connections:
- net FET_1OE: now also R38.1
- net FET_2OE: now also R39.1
- net FET_3OE: now also R40.1
- net FET_4OE: now also R41.1
- net GND: now also U2.3 (VEE), U3.3 (VEE), U4.3 (VEE), U5.3 (VEE)
- new net +3V3: R38.2, R39.2, R40.2, R41.2
