File: PCB/gantry-controller-prototype-DUE/gantry-controller-prototype-DUE.kicad_pcb (KiCad board)
At the start: 4 copper layers, 220 x 130 mm, 130 parts, among them J1 Conn_01x07, M1 D36V50F3, M2 D36V50F5, M3 D36V50F12, M4 Arduino_DUE_Shield_TEMP, Q1 IRLML6346TRPBF, Q2 IRLML6346TRPBF, Q3 IRLML6346TRPBF, Q4 IRLML6346TRPBF, T1 1755736, T10 1755736, T11 1755503, T12 1755503, T13 1740369, T14 1740369, T15 1740369, T16 1740369, T17 1740369, T18 1755574, T19 1755736, T2 1755736, T20 5033981892, T21 5120, T22 5120, T23 5120, T24 5120, T25 5120, T26 5120, T3 1755736, T4 1755736, T5 1755736, T6 1755736, T7 1755736, T8 1755736, T9 1755736, U1 SN74AHCT125RGYR, U2 ZXGD3009E6TA, U3 ZXGD3009E6TA, U4 ZXGD3009E6TA, U5 ZXGD3009E6TA, U6 SHT35-DIS-B2.5KS, U7 74ACT16244DGGR

Commit message: Fab files and edits
made some changes to the circuit, added pullups to OE pins on 74 devices and tied mosfet drivers to GND, added fab files
Parts:
- added R38: RC0402FR-071KL, AVR-KiCAD-Lib-Resistors:R0402, F.Cu at (122.5, 71.5)
- added R39: RC0402FR-071KL, AVR-KiCAD-Lib-Resistors:R0402, F.Cu at (125.2, 66.5)
- added R40: RC0402FR-071KL, AVR-KiCAD-Lib-Resistors:R0402, F.Cu at (113.5, 68.0)
- added R41: RC0402FR-071KL, AVR-KiCAD-Lib-Resistors:R0402, F.Cu at (116.5, 70.8)
- added R42: RC0402FR-071KL, AVR-KiCAD-Lib-Resistors:R0402, F.Cu at (168.5, 132.0)
- added R43: RC0402FR-071KL, AVR-KiCAD-Lib-Resistors:R0402, F.Cu at (168.0, 123.0)
- added R44: RC0402FR-071KL, AVR-KiCAD-Lib-Resistors:R0402, F.Cu at (153.8, 132.0)
- added R45: RC0402FR-071KL, AVR-KiCAD-Lib-Resistors:R0402, F.Cu at (153.5, 123.5)
Connections:
- net /E-Stop and Activity Lights/FET1_DRV renamed /Arduino DUE Connections/FET1_DRV
- net /E-Stop and Activity Lights/FET2_DRV renamed /Arduino DUE Connections/FET2_DRV
- net /E-Stop and Activity Lights/FET3_DRV renamed /Arduino DUE Connections/FET3_DRV
- net /E-Stop and Activity Lights/FET4_DRV renamed /Arduino DUE Connections/FET4_DRV
- net /E-Stop and Activity Lights/FET_1OE renamed /Arduino DUE Connections/FET_1OE
- net /E-Stop and Activity Lights/FET_2OE renamed /Arduino DUE Connections/FET_2OE
- net /E-Stop and Activity Lights/FET_3OE renamed /Arduino DUE Connections/FET_3OE
- net /E-Stop and Activity Lights/FET_4OE renamed /Arduino DUE Connections/FET_4OE
- net /STM32 Board and Connectors/DRV1_DIR renamed /Arduino DUE Connections/DRV1_DIR
- net /STM32 Board and Connectors/DRV1_EN renamed /Arduino DUE Connections/DRV1_EN
- net /STM32 Board and Connectors/DRV1_STEP renamed /Arduino DUE Connections/DRV1_STEP
- net /STM32 Board and Connectors/DRV2_DIR renamed /Arduino DUE Connections/DRV2_DIR
- net /STM32 Board and Connectors/DRV2_EN renamed /Arduino DUE Connections/DRV2_EN
- net /STM32 Board and Connectors/DRV2_STEP renamed /Arduino DUE Connections/DRV2_STEP
- net /STM32 Board and Connectors/DRV3_DIR renamed /Arduino DUE Connections/DRV3_DIR
- net /STM32 Board and Connectors/DRV3_EN renamed /Arduino DUE Connections/DRV3_EN
- net /STM32 Board and Connectors/DRV3_STEP renamed /Arduino DUE Connections/DRV3_STEP
- net /STM32 Board and Connectors/DRV4_DIR renamed /Arduino DUE Connections/DRV4_DIR
- net /STM32 Board and Connectors/DRV4_EN renamed /Arduino DUE Connections/DRV4_EN
- net /STM32 Board and Connectors/DRV4_STEP renamed /Arduino DUE Connections/DRV4_STEP
- net /STM32 Board and Connectors/DRV5_DIR renamed /Arduino DUE Connections/DRV5_DIR
- net /STM32 Board and Connectors/DRV5_EN renamed /Arduino DUE Connections/DRV5_EN
- net /STM32 Board and Connectors/DRV5_STEP renamed /Arduino DUE Connections/DRV5_STEP
- net /STM32 Board and Connectors/END1 renamed /Arduino DUE Connections/END1
- net /STM32 Board and Connectors/END10 renamed /Arduino DUE Connections/END10
- net /STM32 Board and Connectors/END2 renamed /Arduino DUE Connections/END2
- net /STM32 Board and Connectors/END3 renamed /Arduino DUE Connections/END3
- net /STM32 Board and Connectors/END4 renamed /Arduino DUE Connections/END4
- net /STM32 Board and Connectors/END5 renamed /Arduino DUE Connections/END5
- net /STM32 Board and Connectors/END6 renamed /Arduino DUE Connections/END6
- net /STM32 Board and Connectors/END7 renamed /Arduino DUE Connections/END7
- net /STM32 Board and Connectors/END8 renamed /Arduino DUE Connections/END8
- net /STM32 Board and Connectors/END9 renamed /Arduino DUE Connections/END9
- net /STM32 Board and Connectors/UART_CTS renamed /Arduino DUE Connections/UART_CTS
- net /STM32 Board and Connectors/UART_RTS renamed /Arduino DUE Connections/UART_RTS
- net /STM32 Board and Connectors/UART_RX renamed /Arduino DUE Connections/UART_RX
- net /STM32 Board and Connectors/UART_TX renamed /Arduino DUE Connections/UART_TX
- U2 pad 3: Net-(U2-Pad3) -> GND
- U3 pad 3: Net-(U3-Pad3) -> GND
- U4 pad 3: Net-(U4-Pad3) -> GND
- U5 pad 3: Net-(U5-Pad3) -> GND
- U6 pad 2: Net-(U6-Pad2) -> GND
Routing:
- net +3V3: track 22.1 -> 135.6 mm, vias 14 -> 22
- net GND: track 86.0 -> 90.9 mm, vias 90 -> 94
- net Net-(M4-PadD13): track 45.9 -> 48.0 mm
- net /Arduino DUE Connections/FET_2OE: track 18.1 -> 20.0 mm
- net Net-(M4-PadD35): track 70.0 -> 71.2 mm
- net Net-(M4-PadD12): track 38.6 -> 39.8 mm
- net Net-(M4-PadD37): track 77.6 -> 78.6 mm

Commit message: DRC check and gerbers generated, order placed with OSHPark
Parts:
- moved T10 0.50 mm to (46.0, 74.0)
- moved T3 0.50 mm to (46.0, 118.0)
- moved T7 0.50 mm to (46.0, 103.0)
- moved T8 0.50 mm to (46.0, 59.0)
- moved T9 0.50 mm to (46.0, 88.8)
- moved C1 0.25 mm to (57.2, 125.1)
Routing:
- net GND: track 90.9 -> 96.3 mm, vias 94 -> 93
- net /Arduino DUE Connections/FET_3OE: track 46.2 -> 47.2 mm
- net +5V: track 131.4 -> 132.0 mm
- net /Arduino DUE Connections/DRV2_DIR: track 17.6 -> 18.1 mm
- net (no net): vias 1 -> 0
